Commit message: modified urdf for this part and hw0.cpp file, works

File: bin/hw0/resources/rprbot.urdf (robot description, URDF)
Before this commit: robot rprbot, 4 links, 3 joints
Links:
- added link link3, mass 1; visual cylinder length=2.0 radius=0.03; visual sphere radius=0.09
- link link2: mass 1 -> 0.01; geometry visual cylinder length=0 radius=0.03
Joints:
- added joint j3: type prismatic, parent link2, child link3, origin xyz=0 0 0 rpy=0 0 0, axis 0 0 1, limit lower=-2.967 upper=2.967 effort=176 velocity=1.7104
